File: PCB/EAGLE/FETbox_rev0_PCB.brd (EAGLE design)
At the start: 120.6 x 43.3 mm, 40 parts, among them J4 ACCESSORY_HEADER, Q1 IRF520, Q2 IRF520, Q3 IRF520, Q4 IRF520, Q5 IRF520, U1 CL13845G, U2 CL13845G, U3 CL13845G, U4 CL13845G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

Commit message: sketch improved, fetbox lid, schematics
Parts:
- Q1, Q2, Q3, Q4, Q5: value IRF520 -> FQP30N06L; device transistor-power:TO220BV -> PerfusionHardwareController:TO220
