File: PCB/EAGLE/FETbox_rev0_PCB.sch (EAGLE design)
At the start: 40 parts, among them J4 ACCESSORY_HEADER, Q1 IRF520, Q2 IRF520, Q3 IRF520, Q4 IRF520, Q5 IRF520, U1 CL13845G, U2 CL13845G, U3 CL13845G, U4 CL13845G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

Commit message: sketch improved, fetbox lid, schematics
Parts:
- Q1, Q2, Q3, Q4, Q5: value IRF520 -> FQP30N06L; device transistor-power:IRF520 -> PerfusionHardwareController:FQP30N06L
Other:
- moved on the sheet: H3
Changed lines of the file:
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@@
 </groups>
 <parts>
-<part name="Q1" library="transistor-power" library_urn="urn:adsk.eagle:library:400" deviceset="IRF520" device="" package3d_urn="urn:adsk.eagle:package:29484/3"/>
+<part name="Q1" library="PerfusionHardwareController" library_urn="urn:adsk.eagle:library:24117063" deviceset="FQP30N06L" device="" package3d_urn="urn:adsk.eagle:package:29484/3"/>
 <part name="R1" library="rcl" library_urn="urn:adsk.eagle:library:334" deviceset="R-EU_" device="0207/10" package3d_urn="urn:adsk.eagle:package:23491/2" value="100"/>
 <part name="D1" library="diode" library_urn="urn:adsk.eagle:library:210" deviceset="1N4004" device="" package3d_urn="urn:adsk.eagle:package:43336/1"/>
@@
 <part name="R2" library="rcl" library_urn="urn:adsk.eagle:library:334" deviceset="R-EU_" device="0207/10" package3d_urn="urn:adsk.eagle:package:23491/2" value="10K"/>
 <part name="U1" library="PerfusionHardwareController" library_urn="urn:adsk.eagle:library:24117063" deviceset="CL13845G" device="" package3d_urn="urn:adsk.eagle:package:24117076/2"/>
-<part name="Q2" library="transistor-power" library_urn="urn:adsk.eagle:library:400" deviceset="IRF520" device="" package3d_urn="urn:adsk.eagle:package:29484/3"/>
+<part name="Q2" library="PerfusionHardwareController" library_urn="urn:adsk.eagle:library:24117063" deviceset="FQP30N06L" device="" package3d_urn="urn:adsk.eagle:package:29484/3"/>
 <part name="R3" library="rcl" library_urn="urn:adsk.eagle:library:334" deviceset="R-EU_" device="0207/10" package3d_urn="urn:adsk.eagle:package:23491/2" value="100"/>
 <part name="D2" library="diode" library_urn="urn:adsk.eagle:library:210" deviceset="1N4004" device="" package3d_urn="urn:adsk.eagle:package:43336/1"/>
@@
 <part name="R4" library="rcl" library_urn="urn:adsk.eagle:library:334" deviceset="R-EU_" device="0207/10" package3d_urn="urn:adsk.eagle:package:23491/2" value="10K"/>
 <part name="U2" library="PerfusionHardwareController" library_urn="urn:adsk.eagle:library:24117063" deviceset="CL13845G" device="" package3d_urn="urn:adsk.eagle:package:24117076/2"/>
-<part name="Q3" library="transistor-power" library_urn="urn:adsk.eagle:library:400" deviceset="IRF520" device="" package3d_urn="urn:adsk.eagle:package:29484/3"/>
+<part name="Q3" library="PerfusionHardwareController" library_urn="urn:adsk.eagle:library:24117063" deviceset="FQP30N06L" device="" package3d_urn="urn:adsk.eagle:package:29484/3"/>
 <part name="R5" library="rcl" library_urn="urn:adsk.eagle:library:334" deviceset="R-EU_" device="0207/10" package3d_urn="urn:adsk.eagle:package:23491/2" value="100"/>
 <part name="D3" library="diode" library_urn="urn:adsk.eagle:library:210" deviceset="1N4004" device="" package3d_urn="urn:adsk.eagle:package:43336/1"/>
@@
 <part name="R6" library="rcl" library_urn="urn:adsk.eagle:library:334" deviceset="R-EU_" device="0207/10" package3d_urn="urn:adsk.eagle:package:23491/2" value="10K"/>
 <part name="U3" library="PerfusionHardwareController" library_urn="urn:adsk.eagle:library:24117063" deviceset="CL13845G" device="" package3d_urn="urn:adsk.eagle:package:24117076/2"/>
-<part name="Q4" library="transistor-power" library_urn="urn:adsk.eagle:library:400" deviceset="IRF520" device="" package3d_urn="urn:adsk.eagle:package:29484/3"/>
+<part name="Q4" library="PerfusionHardwareController" library_urn="urn:adsk.eagle:library:24117063" deviceset="FQP30N06L" device="" package3d_urn="urn:adsk.eagle:package:29484/3"/>
 <part name="R7" library="rcl" library_urn="urn:adsk.eagle:library:334" deviceset="R-EU_" device="0207/10" package3d_urn="urn:adsk.eagle:package:23491/2" value="100"/>
 <part name="D4" library="diode" library_urn="urn:adsk.eagle:library:210" deviceset="1N4004" device="" package3d_urn="urn:adsk.eagle:package:43336/1"/>
@@
 <part name="R8" library="rcl" library_urn="urn:adsk.eagle:library:334" deviceset="R-EU_" device="0207/10" package3d_urn="urn:adsk.eagle:package:23491/2" value="10K"/>
 <part name="U4" library="PerfusionHardwareController" library_urn="urn:adsk.eagle:library:24117063" deviceset="CL13845G" device="" package3d_urn="urn:adsk.eagle:package:24117076/2"/>
-<part name="Q5" library="transistor-power" library_urn="urn:adsk.eagle:library:400" deviceset="IRF520" device="" package3d_urn="urn:adsk.eagle:package:29484/3"/>
+<part name="Q5" library="PerfusionHardwareController" library_urn="urn:adsk.eagle:library:24117063" deviceset="FQP30N06L" device="" package3d_urn="urn:adsk.eagle:package:29484/3"/>
 <part name="R9" library="rcl" library_urn="urn:adsk.eagle:library:334" deviceset="R-EU_" device="0207/10" package3d_urn="urn:adsk.eagle:package:23491/2" value="100"/>
 <part name="D5" library="diode" library_urn="urn:adsk.eagle:library:210" deviceset="1N4004" device="" package3d_urn="urn:adsk.eagle:package:43336/1"/>
@@
 <instance part="R1" gate="G$1" x="88.9" y="119.38" smashed="yes" grouprefs="OUTPUT1">
 <attribute name="NAME" x="85.09" y="120.8786" size="1.778" layer="95"/>
-<attribute name="VALUE" x="85.09" y="116.078" size="1.778" layer="96"/>
 </instance>
 <instance part="D1" gate="1" x="99.06" y="132.08" smashed="yes" rot="R90" grouprefs="OUTPUT1">
@@
 <instance part="R3" gate="G$1" x="137.16" y="119.38" smashed="yes" grouprefs="OUTPUT2">
 <attribute name="NAME" x="133.35" y="120.8786" size="1.778" layer="95"/>
-<attribute name="VALUE" x="133.35" y="116.078" size="1.778" layer="96"/>
 </instance>
 <instance part="D2" gate="1" x="147.32" y="132.08" smashed="yes" rot="R90" grouprefs="OUTPUT2">
@@
 <instance part="R5" gate="G$1" x="185.42" y="119.38" smashed="yes" grouprefs="OUTPUT3">
 <attribute name="NAME" x="181.61" y="120.8786" size="1.778" layer="95"/>
-<attribute name="VALUE" x="181.61" y="116.078" size="1.778" layer="96"/>
 </instance>
 <instance part="D3" gate="1" x="195.58" y="132.08" smashed="yes" rot="R90" grouprefs="OUTPUT3">
@@
 <instance part="R7" gate="G$1" x="137.16" y="68.58" smashed="yes" grouprefs="OUTPUT4">
 <attribute name="NAME" x="133.35" y="70.0786" size="1.778" layer="95"/>
-<attribute name="VALUE" x="133.35" y="65.278" size="1.778" layer="96"/>
 </instance>
 <instance part="D4" gate="1" x="147.32" y="81.28" smashed="yes" rot="R90" grouprefs="OUTPUT4">
@@
 <instance part="R9" gate="G$1" x="187.96" y="68.58" smashed="yes" grouprefs="OUTPUT5">
 <attribute name="NAME" x="184.15" y="70.0786" size="1.778" layer="95"/>
-<attribute name="VALUE" x="184.15" y="65.278" size="1.778" layer="96"/>
 </instance>
 <instance part="D5" gate="1" x="198.12" y="81.28" smashed="yes" rot="R90" grouprefs="OUTPUT5">
@@
 <attribute name="NAME" x="223.012" y="150.4442" size="1.778" layer="95"/>
 </instance>
-<instance part="H3" gate="G$1" x="22.86" y="35.56" smashed="yes">
-<attribute name="NAME" x="24.892" y="36.1442" size="1.778" layer="95"/>
+<instance part="H3" gate="G$1" x="15.24" y="48.26" smashed="yes">
+<attribute name="NAME" x="17.272" y="48.8442" size="1.778" layer="95"/>
 </instance>
 <instance part="H4" gate="G$1" x="215.9" y="43.18" smashed="yes">
